File: design/pyros.kicad_sch (KiCad schematic)
At the start: 19 parts, among them J3 Screw_Terminal_01x06, U10 VN7050ASTR, U11 VN7050ASTR, U9 VN7050ASTR

Commit message: PCB 1.1 old regulator
Parts:
- D4: mfn (none) -> PZU3.0B2,115
- D5, D6, D8: mfn (none) -> CG0603MLC-24LEA
- F1, F2, F3: mfn (none) -> 1210L150/16WR
Changed lines of the file:
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@@
+      (effects (font (size 1.27 1.27)) hide)
+    )
+    (property "mfn" " CG0603MLC-24LEA" (at 130.81 107.95 90)
       (effects (font (size 1.27 1.27)) hide)
     )
@@
       (effects (font (size 1.27 1.27)) hide)
     )
+    (property "Field4" "" (at 137.16 78.74 90)
+      (effects (font (size 1.27 1.27)) hide)
+    )
+    (property "mfn" " 1210L150/16WR " (at 137.16 78.74 0)
+      (effects (font (size 1.27 1.27)) hide)
+    )
     (pin "1")
     (pin "2")
@@
       (effects (font (size 1.27 1.27)) hide)
     )
+    (property "mfn" " CG0603MLC-24LEA" (at 130.81 83.82 90)
+      (effects (font (size 1.27 1.27)) hide)
+    )
     (pin "1")
     (pin "2")
@@
     )
     (property "Datasheet" "~" (at 137.16 102.87 0)
+      (effects (font (size 1.27 1.27)) hide)
+    )
+    (property "mfn" " 1210L150/16WR " (at 137.16 102.87 90)
       (effects (font (size 1.27 1.27)) hide)
     )
@@
     )
     (property "Datasheet" "~" (at 109.22 58.42 90)
+      (effects (font (size 1.27 1.27)) hide)
+    )
+    (property "mfn" " PZU3.0B2,115 " (at 109.22 58.42 90)
       (effects (font (size 1.27 1.27)) hide)
     )
@@
       (effects (font (size 1.27 1.27)) hide)
     )
+    (property "mfn" " PZU3.0B2,115 " (at 109.22 106.68 90)
+      (effects (font (size 1.27 1.27)) hide)
+    )
     (pin "1")
     (pin "2")
@@
       (effects (font (size 1.27 1.27)) hide)
     )
+    (property "mfn" " 1210L150/16WR " (at 137.16 54.61 90)
+      (effects (font (size 1.27 1.27)) hide)
+    )
     (pin "1")
     (pin "2")
@@
       (effects (font (size 1.27 1.27)) hide)
     )
+    (property "mfn" " PZU3.0B2,115 " (at 109.22 82.55 90)
+      (effects (font (size 1.27 1.27)) hide)
+    )
     (pin "1")
     (pin "2")
@@
       (effects (font (size 1.27 1.27)) hide)
     )
+    (property "mfn" " CG0603MLC-24LEA" (at 130.81 59.69 90)
+      (effects (font (size 1.27 1.27)) hide)
+    )

Commit message: PCB v1.1
Parts:
- added R11 (x3): 10k, Resistor_SMD:R_0603_1608Metric, symbol Device:R_Small
- D4: footprint Diode_SMD:D_0603_1608Metric -> Diode_SMD:D_SOD-323_HandSoldering
Connections:
- net Earth: now also R11.2, R11.2, R11.2
- net PYRO1_EN: now also R11.1
- net PYRO2_EN: now also R11.1
- net PYRO3_EN: now also R11.1

Commit message: v1.2
Parts:
- R11, R3, R4: renamed from R5; value 47k -> 3k
- R12, R17, R5: renamed from R11; value 47k -> 3k
- renumbered D4 to D3, D4 to D7, J3 to J7, R11 to R28, R11 to R29, R11 to R30
Other:
- note removed: "1uA back current"
